File: weather-dash.kicad_pcb (KiCad board)
At the start: 11 copper layers, 59.5 x 43.5 mm, 7 parts, among them J1 Conn_01x02_Pin, J3 Conn_01x03_Socket, SW1 SW_Push, U1 WEMOS_C3_Mini, U2 TFT_ST7735_SD

Commit message: updates
Parts:
- added D1: 1N5817, Diode_THT:D_DO-41_SOD81_P7.62mm_Horizontal, F.Cu at (28.2, 54.5)
- added G***: LOGO, LOGO, B.Cu at (62.5, 30.5)
- added R3: 10K, Resistor_THT:R_Axial_DIN0207_L6.3mm_D2.5mm_P7.62mm_Horizontal, F.Cu at (64.0, 67.3)
- added SW2: SW_SPDT, Connector_JST:JST_PH_B2B-PH-K_1x02_P2.00mm_Vertical, B.Cu at (31.5, 42.5)
- added SW3: SW_Push, Button_Switch_THT:SW_PUSH_6mm_H4.3mm, F.Cu at (67.8, 62.5)
- added U3: ~, asylum-weather:TP4056, B.Cu at (29.5, 60.0)
- J3: footprint Connector_PinSocket_2.54mm:PinSocket_1x03_P2.54mm_Vertical -> asylum-weather:DHT11
- R2: moved to F.Cu
- U1: footprint Module:WEMOS_D1_mini_light -> asylum-weather:WEMOS_C3_mini
- moved SW1 47.8 mm to (22.8, 62.5)
- moved R2 38.5 mm to (41.3, 60.0), turned to 180 degrees
- moved U1 19.6 mm to (57.1, 49.4), turned to 180 degrees
- moved J1 15.3 mm to (40.5, 42.5), turned to 180 degrees
- moved J3 2.55 mm to (25.5, 27.0)
- moved R1 1.40 mm to (24.5, 41.7)
Connections:
- J1 pad 1: GND -> BAT-
- J1 pad 2: VBUS -> BAT+
- R2 pad 1: BTN -> BTN1
- SW1 pad 1: BTN -> BTN1
- U1 pad 2: TFT_EN -> SD_CS
- U1 pad 4: SD_CS -> DHT11
- U1 pad 5: BTN -> TFT_EN
- U1 pad 6: DHT11 -> BTN1
- U1 pad 7: unconnected-(U1-IO5-Pad7) -> BTN2
Routing:
- net BTN1: track 0.00 -> 51.6 mm
- net BTN: track 35.7 -> 0.00 mm
- net BAT+: track 0.00 -> 22.5 mm
- net +3.3V: track 68.5 -> 88.0 mm
- net BTN2: track 0.00 -> 19.0 mm
- net TFT_EN: track 40.5 -> 57.8 mm
- net BAT-: track 0.00 -> 16.7 mm
- net MISO: track 22.0 -> 5.99 mm
- net DHT11: track 36.6 -> 52.4 mm
- net TFT_DC: track 44.4 -> 29.1 mm
- net Net-(D1-A): track 0.00 -> 14.2 mm
- net Net-(D1-K): track 0.00 -> 12.5 mm
- net VBUS: track 40.2 -> 30.7 mm
- net SD_CS: track 17.4 -> 8.53 mm
- net TFT_CS: track 42.5 -> 34.3 mm
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Other:
- board size 59.5 x 43.5 mm -> 61 x 45.5 mm
- board text added: "@grimsteel"
- board text added: "Weather Dash"
- board text added: "v0.2"
- board text removed: "BAT"

Commit message: some changes
idk what they are
Parts:
- moved J3 2.98 mm to (28.5, 27.0)
- moved G*** 2.50 mm to (65.0, 30.5)
Routing:
- net DHT11: track 52.4 -> 49.9 mm
- net +3.3V: track 88.0 -> 90.4 mm
Other:
- board text added: "JLCJLCJLCJLC"

Commit message: more pcb changes
Parts:
- removed R2, R3: 10K, Resistor_THT:R_Axial_DIN0207_L6.3mm_D2.5mm_P7.62mm_Horizontal
- added BZ1: Buzzer, Buzzer_Beeper:Buzzer_12x9.5RM7.6, B.Cu at (39.5, 36.2)
- SW2: value SW_SPDT -> SW_SPST
- U1: value WEMOS_C3_Mini -> WEMOS_S2_Mini; footprint asylum-weather:WEMOS_C3_mini -> asylum-weather:WEMOS_S2_Mini
- moved J1 7.49 mm to (37.2, 49.2), turned to 0 degrees
- moved SW2 6.97 mm to (29.8, 49.2), turned to 0 degrees
- moved SW1 2.51 mm to (20.2, 62.8)
- moved D1 2.30 mm to (27.7, 56.8)
- moved J3 2.00 mm to (30.5, 27.0)
- moved G*** 2.00 mm to (67.0, 30.5)
- moved U1 1.75 mm to (55.4, 50.0)
- moved U3 1.12 mm to (28.5, 60.5)
- moved SW3 0.75 mm to (67.8, 63.2)
Connections:
- SW2 pad 1: VBUS -> Net-(D1-K)
- SW2 pad 2: Net-(D1-K) -> VBUS
- U1 pad 10: GND -> unconnected-(U1-IO2-Pad10)
- U1 pad 11: SCK -> unconnected-(U1-IO4-Pad11)
- U1 pad 12: MOSI -> unconnected-(U1-IO6-Pad12)
- U1 pad 13: TFT_DC -> unconnected-(U1-IO8-Pad13)
- U1 pad 14: TFT_CS -> unconnected-(U1-IO10/CS0-Pad14)
- U1 pad 16: unconnected-(U1-TX-Pad16) -> BTN2
- U1 pad 2: SD_CS -> unconnected-(U1-IO3-Pad2)
- U1 pad 3: MISO -> unconnected-(U1-IO5-Pad3)
- U1 pad 4: DHT11 -> unconnected-(U1-IO7-Pad4)
- U1 pad 5: TFT_EN -> unconnected-(U1-IO9-Pad5)
- U1 pad 6: BTN1 -> unconnected-(U1-IO11/MOSI-Pad6)
- U1 pad 7: BTN2 -> unconnected-(U1-IO12/SCK-Pad7)
- U1 pad 9: VBUS -> SD_CS
Routing:
- net TFT_EN: track 57.8 -> 29.0 mm
- net DHT11: track 49.9 -> 21.6 mm
- net MISO: track 5.99 -> 29.6 mm
- net BTN1: track 51.6 -> 38.1 mm
- net BUZ: track 0.00 -> 10.8 mm
- net VBUS: track 30.7 -> 21.4 mm
- net BAT-: track 16.7 -> 7.97 mm
- net BTN2: track 19.0 -> 11.5 mm
- net SCK: track 62.1 -> 56.1 mm
- net BAT+: track 22.5 -> 17.0 mm
- net +3.3V: track 90.4 -> 85.6 mm
- net TFT_CS: track 34.3 -> 38.8 mm
- net MOSI: track 60.7 -> 57.0 mm
- net Net-(D1-K): track 12.5 -> 9.10 mm
- net SD_CS: track 8.53 -> 10.4 mm
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Other:
- board size 61 x 45.5 mm -> 61 x 46 mm
- board text added: "v0.4"
- board text removed: "v0.2"
