File: weather-dash.kicad_sch (KiCad schematic)
At the start: 7 parts, among them J1 Conn_01x02_Pin, J3 Conn_01x03_Socket, SW1 SW_Push, U1 WEMOS_C3_Mini, U2 TFT_ST7735_SD

Commit message: updates
Parts:
- added D1: 1N5817, Diode_THT:D_DO-41_SOD81_P7.62mm_Horizontal, symbol Device:D
- added R3: 10K, Resistor_THT:R_Axial_DIN0207_L6.3mm_D2.5mm_P7.62mm_Horizontal, symbol Device:R
- added SW2: SW_SPDT, Connector_JST:JST_PH_B2B-PH-K_1x02_P2.00mm_Vertical, symbol Switch:SW_SPDT
- added SW3: SW_Push, Button_Switch_THT:SW_PUSH_6mm_H4.3mm, symbol Switch:SW_Push
- added U3: ~, asylum-weather:TP4056, symbol asylum-weather:TP4056
- J3: footprint Connector_PinSocket_2.54mm:PinSocket_1x03_P2.54mm_Vertical -> asylum-weather:DHT11
- U1: footprint Module:WEMOS_D1_mini_light -> asylum-weather:WEMOS_C3_mini
Connections:
- net +3.3V: now also R3.2
- net DHT11: now also U1.4 (IO1); no longer U1.6 (IO4)
- net GND: now also SW3.2, U3.3 (OUT-); no longer J1.1 (Pin_1)
- net SD_CS: now also U1.2 (IO3); no longer U1.4 (IO1)
- net TFT_EN: now also U1.5 (IO0); no longer U1.2 (IO3)
- net VBUS: now also SW2.1 (A); no longer J1.2 (Pin_2)
- net BTN2: now reaches U1.7 (IO5)
- net BTN2: now also R3.1, SW3.1
- net BTN renamed BTN1
- net BTN1: now also U1.6 (IO4); no longer U1.5 (IO0)
- new net: D1.1 (K), SW2.2 (B)
- new net: D1.2 (A), U3.2 (OUT+)
- new net BAT+: J1.2 (Pin_2), U3.0 (BAT+)
- new net BAT-: J1.1 (Pin_1), U3.1 (BAT-)
- no-connect marks 3 -> 6
Other:
- note added: "BUTTON 1"
- note added: "BUTTON 2"
- note added: "POWER + CHARGING"
- note removed: "BUTTON"
- moved on the sheet: J1, J3, R2, SW1, U1

Commit message: some changes
idk what they are
Parts:
- SW2: symbol Switch:SW_SPDT -> Switch:SW_SPST
Connections:
- no-connect marks 6 -> 5
Changed lines of the file:
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@@
-	)
-	(no_connect
-		(at 91.44 74.93)
 	)
 	(no_connect
@@
 		(on_board yes)
 		(dnp no)
-		(fields_autoplaced yes)
 		(property "Reference" "J1"
 			(at 69.215 64.77 0)
@@
 		)
 		(property "Value" "Conn_01x02_Pin"
-			(at 69.215 67.31 0)
+			(at 68.58 67.31 0)
 			(effects
 				(font
@@
 	(symbol
 		(lib_id "power:VBUS")
-		(at 91.44 69.85 90)
+		(at 91.44 72.39 90)
 		(unit 1)
 		(exclude_from_sim no)
@@
 		(dnp no)
 		(property "Reference" "#PWR012"
-			(at 95.25 69.85 0)
+			(at 95.25 72.39 0)
 			(effects
 				(font
@@
 		)
 		(property "Value" "VBUS"
-			(at 91.186 67.818 90)
+			(at 91.186 70.358 90)
 			(effects
 				(font
@@
 		)
 		(property "Footprint" ""
-			(at 91.44 69.85 0)
+			(at 91.44 72.39 0)
 			(effects
 				(font
@@
 		)
 		(property "Datasheet" ""
-			(at 91.44 69.85 0)
+			(at 91.44 72.39 0)
 			(effects
 				(font
@@
 		)
 		(property "Description" "Power symbol creates a global label with name \"VBUS\""
-			(at 91.44 69.85 0)
+			(at 91.44 72.39 0)
 			(effects
 				(font
@@
 		(on_board yes)
 		(dnp no)
-		(fields_autoplaced yes)
 		(property "Reference" "D1"
 			(at 107.95 66.04 0)
@@
 		)
 		(property "Value" "1N5817"
-			(at 107.95 68.58 0)
+			(at 108.204 68.834 0)
 			(effects
 				(font
@@
 	)
 	(symbol
-		(lib_id "Switch:SW_SPDT")
+		(lib_id "Switch:SW_SPST")
 		(at 96.52 72.39 0)
-		(mirror y)
 		(unit 1)
 		(exclude_from_sim no)
@@
 		)
 		(property "Datasheet" "~"
-			(at 96.52 80.01 0)
-			(effects
-				(font
-					(size 1.27 1.27)
-				)
-				(hide yes)
-			)
-		)
-		(property "Description" "Switch, single pole double throw"
 			(at 96.52 72.39 0)
 			(effects
@@
 			)
 		)
+		(property "Description" "Single Pole Single Throw (SPST) switch"
+			(at 96.52 72.39 0)
+			(effects
+				(font
+					(size 1.27 1.27)
+				)
+				(hide yes)
+			)
+		)
 		(pin "1"
 		)
-		(pin "3"
-		)
 		(pin "2"

Commit message: more pcb changes
Parts:
- removed R2, R3: 10K, Resistor_THT:R_Axial_DIN0207_L6.3mm_D2.5mm_P7.62mm_Horizontal, symbol Device:R
- removed U1: WEMOS_C3_Mini, asylum-weather:WEMOS_C3_mini, symbol wemos_c3_mini:WEMOS_C3_mini
- added BZ1: Buzzer, Buzzer_Beeper:Buzzer_12x9.5RM7.6, symbol Device:Buzzer
- added U1: WEMOS_S2_Mini, asylum-weather:WEMOS_S2_Mini, symbol asylum-weather:WEMOS_S2_Mini
- SW2: value SW_SPDT -> SW_SPST
Connections:
- net +3.3V: now also U1.8 (3V3)
- net BTN1: now also U1.22 (IO17)
- net BTN2: now also U1.16 (IO14)
- net DHT11: now also U1.25 (IO39)
- net GND: now also BZ1.2 (-), U1.23 (GND)
- net MISO: now also U1.26 (IO37/MISO)
- net MOSI: now also U1.27 (IO35/MOSI)
- net SCK: now also U1.19 (IO36/SCK)
- net SD_CS: now also U1.9 (IO1)
- net TFT_CS: now also U1.20 (IO34/CS0)
- net TFT_DC: now also U1.28 (IO33)
- net TFT_EN: now also U1.18 (IO38)
- net VBUS: now also SW2.2 (B), U1.32 (VBUS); no longer SW2.1 (A)
- net at D1.1 (K): now also SW2.1 (A); no longer SW2.2 (B)
- new net BUZ: BZ1.1 (+), U1.17 (IO40)
Other:
- note added: "BUZZER"
- moved on the sheet: D1, J1, J3, R1, SW1, SW2, SW3, U2, U3
